File: doc/pi-pico-pcb/proto-pi-pico-pcb/Normal_Port_Sheet.kicad_sch (KiCad schematic)
At the start: 1 part

Commit message: added flash memory
Other:
- company: (none) -> PROTO
Changed lines of the file:
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@@
 (kicad_sch (version 20211123) (generator eeschema)
   (paper "A4")
+  (title_block
+    (date "2025-09-09")
+    (rev "1")
+    (company "PROTO")
+    (comment 1 "Author: Carston Wiebe")
+  )
   (no_connect (at 136.525 107.95))
   (no_connect (at 136.525 110.49))
